File: hardware/pcb/controller_board/Pico2Breakout/Pico2Breakout.kicad_sch (KiCad schematic)
At the start: 5 parts, among them J11 UART, J19 Screw_Terminal_01x02, J20 Screw_Terminal_01x02, J21 Screw_Terminal_01x02

Commit message: working board update
Connections:
- net GNDA is gone; now on net GND2: J11.1 (Pin_1)
- no-connect marks 1 -> 5
Changed lines of the file:
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@@
+	)
+	(no_connect
+		(at 189.23 88.9)
+	)
+	(no_connect
+		(at 189.23 104.14)
 	)
 	(no_connect
 		(at 166.37 43.18)
+	)
+	(no_connect
+		(at 143.51 58.42)
+	)
+	(no_connect
+		(at 143.51 60.96)
 	)
 	(wire
@@
 			)
 		)
-		(property "Value" "GNDA"
+		(property "Value" "GND2"
 			(at 144.78 45.212 0)
 			(effects
