File: hardware/pcb/controller_board/RP2350B_breakout/RP2350B_breakout.kicad_sch (KiCad schematic)
At the start: 38 parts, among them J1 USB_B_Micro, J4 SM03B-SRSS-TB, SW1 SW_Push, SW2 SW_Push, U1 RP2350_80QFN, U2 NCP1117-3.3_SOT223, U3 W25Q128JVS, Y1 ABM8-272-T3

Commit message: KiCAD files for 6 axis RP2350B board
Parts:
- added D29, D30: LED, LED_SMD:LED_0805_2012Metric, symbol Device:LED
- added D8, D9: PMEG4010EP,115, Diode_SMD:D_SOD-128, symbol Diode:PMEG4010EH
- added H1, H2, H3, H4, H5, H6: MountingHole, MountingHole:MountingHole_3.2mm_M3_ISO7380, symbol Mechanical:MountingHole
- added J3: Conn_01x02, Connector_JST:JST_NV_B02P-NV_1x02_P5.00mm_Vertical, symbol Connector_Generic:Conn_01x02
- added J48: UART, Connector_PinHeader_2.54mm:PinHeader_1x04_P2.54mm_Vertical, symbol Connector:Conn_01x04_Pin
- added J49: aux1, Connector_PinHeader_2.54mm:PinHeader_1x04_P2.54mm_Vertical, symbol Connector:Conn_01x04_Pin
- added J50: aux2, Connector_PinHeader_2.54mm:PinHeader_1x04_P2.54mm_Vertical, symbol Connector:Conn_01x04_Pin
- added R78, R79, R80, R81, R82, R85: 4.7kOhm, Resistor_SMD:R_0805_2012Metric, symbol Device:R
- added R83, R84, R86, R87, R88, R89, R90, R91: 470, Resistor_SMD:R_0805_2012Metric, symbol Device:R
- added U28, U29: TLP291-4_TP_E_, TLP291-4_TP_E_:SOIC127P700X229-16N, symbol TLP291-4_TP_E_:TLP291-4_TP_E_
- renumbered J4 to J2
Connections:
- net +3V3: now also J48.4 (Pin_4), J49.4 (Pin_4), J50.4 (Pin_4), R78.2, R79.2, R80.2, R81.2, R82.2, R83.1, R85.2
- net GND: now also D29.1 (K), D30.1 (K), J3.2 (Pin_2), J48.1 (Pin_1), J49.1 (Pin_1), J50.1 (Pin_1), U28.11, U28.13, U28.15, U28.2, U28.4, U28.6, U28.8, U28.9, U29.13, U29.15, U29.2, U29.4
- net GPIO0: now also J48.3 (Pin_3)
- net GPIO1: now also J48.2 (Pin_2)
- net GPIO10: now also R81.1, U28.16
- net GPIO11: now also R78.1, U28.14
- net GPIO12: now also R79.1, U28.12
- net GPIO13: now also R80.1, U28.10
- net GPIO14: now also R85.1, U29.16
- net GPIO15: now also R82.1, U29.14
- net GPIO41_ADC1: now also J49.2 (Pin_2)
- net GPIO42_ADC2: now also J49.3 (Pin_3)
- net GPIO43_ADC3: now also J50.2 (Pin_2)
- net GPIO44_ADC4: now also J50.3 (Pin_3)
- net GPIO47_ADC7: now also R84.1
- net VBUS: no longer names the net of C1.1, U2.3 (VI)
- net VBUS: now also D8.1 (K), D9.1 (K); no longer J1.1 (VBUS)
- new net: D8.2 (A), J1.1 (VBUS)
- new net: R86.1, U28.1
- new net: R87.1, U28.3
- new net: R88.1, U28.5
- new net: R89.1, U28.7
- new net: D29.2 (A), R83.2
- new net: D30.2 (A), R84.2
- new net: R90.1, U29.1
- new net: R91.1, U29.3
- new net +48V: J3.1 (Pin_1)
- new net +5V: D9.2 (A)
- new net A_err: R89.2
- new net B_err: R90.2
- new net C_err: R91.2
- new net X_err: R86.2
- new net Y_err: R87.2
- new net Z_err: R88.2
- no-connect marks 1 -> 11
Other:
- sheet axis renamed axis_1
- added sheet 12V_converter (12V_converter.kicad_sch)
- added sheet 5V_converter (5V_converter.kicad_sch)
- added sheet Homing_Estop (Inputs_homingEstop.kicad_sch)
- added sheet PWMout_1 (pwm_outputs.kicad_sch)
- added sheet PWMout_2 (pwm_outputB.kicad_sch)
- added sheet axis_2 (axis.kicad_sch)
- added sheet axis_3 (axis.kicad_sch)
- added sheet axis_4 (axis.kicad_sch)
- added sheet axis_5 (axis.kicad_sch)
- added sheet axis_6 (axis.kicad_sch)
- added sheet outputRelay (output_relays.kicad_sch)
- sheet axis_1 ports: added err; removed none
- note added: "3V3_conveter"
- moved on the sheet: C1, C10, C11, C12, C13, C14, C15, C16, C17, C18, C19, C2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
